File: hardware/rack-ui-pcb/rack-ui-pcb.kicad_sch (KiCad schematic)
At the start: 53 parts, among them J1 IO, J2 Conn_ARM_SWD_TagConnect_TC203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, Q1 BC817-40W, Q2 BC817-40W, SW1 EC11E18244A5, U1 PY32F002AW15U, U2 HT42B534-2, U3 ME6211C33M5G-N

Commit message: updated LCSC# field, added PCB text
Parts:
- J1: LCSC C109410 -> C9136; LCSC Part C109410 -> C9136
Changed lines of the file:
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@@
 			)
 		)
-		(property "LCSC" "C109410"
+		(property "LCSC" "C9136"
 			(at 44.45 39.37 0)
 			(hide yes)
@@
 			)
 		)
-		(property "LCSC Part" "C109410"
+		(property "LCSC Part" "C9136"
 			(at 44.45 39.37 0)
 			(hide yes)
